File: HW/ni.sch (EAGLE design)
At the start: 71 parts, among them IC1 FAN3100TSX, IC2 STM32G071CBU6, IC3 MIC5504-3.3YM5-TR, Q1 FQD12N20L, Q10 CPH3461, Q11 CPH3461, Q12 CPH3461, Q13 BF821SMD, Q14 CPH3461, Q15 BF821SMD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

Commit message: HW_values added
Parts:
- C3, C8: value (none) -> 4.3p
- R16: value (none) -> 15k
Changed lines of the file:
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@@
 <part name="FRAME2" library="frames" library_urn="urn:adsk.eagle:library:229" deviceset="A4L-LOC" device=""/>
 <part name="IC2" library="STM32G071CBU6" library_urn="urn:adsk.eagle:library:13357853" deviceset="STM32G071CBU6" device="" package3d_urn="urn:adsk.eagle:package:13357856/2"/>
-<part name="C3" library="rcl" library_urn="urn:adsk.eagle:library:334" deviceset="C-EU" device="C0402" package3d_urn="urn:adsk.eagle:package:23626/2"/>
+<part name="C3" library="rcl" library_urn="urn:adsk.eagle:library:334" deviceset="C-EU" device="C0402" package3d_urn="urn:adsk.eagle:package:23626/2" value="4.3p"/>
 <part name="C4" library="rcl" library_urn="urn:adsk.eagle:library:334" deviceset="C-EU" device="C1206" package3d_urn="urn:adsk.eagle:package:23618/2" value="47u"/>
 <part name="C5" library="rcl" library_urn="urn:adsk.eagle:library:334" deviceset="C-EU" device="C1206" package3d_urn="urn:adsk.eagle:package:23618/2" value="47u"/>
@@
 <part name="GND9" library="supply1" library_urn="urn:adsk.eagle:library:371" deviceset="GND" device=""/>
 <part name="X1" library="crystal" library_urn="urn:adsk.eagle:library:204" deviceset="FC-12M" device="" package3d_urn="urn:adsk.eagle:package:12123/1"/>
-<part name="C8" library="rcl" library_urn="urn:adsk.eagle:library:334" deviceset="C-EU" device="C0402" package3d_urn="urn:adsk.eagle:package:23626/2"/>
+<part name="C8" library="rcl" library_urn="urn:adsk.eagle:library:334" deviceset="C-EU" device="C0402" package3d_urn="urn:adsk.eagle:package:23626/2" value="4.3p"/>
 <part name="GND10" library="supply1" library_urn="urn:adsk.eagle:library:371" deviceset="GND" device=""/>
 <part name="GND11" library="supply1" library_urn="urn:adsk.eagle:library:371" deviceset="GND" device=""/>
@@
 <part name="P+12" library="supply1" library_urn="urn:adsk.eagle:library:371" deviceset="+5V" device=""/>
 <part name="R15" library="rcl" library_urn="urn:adsk.eagle:library:334" deviceset="R-EU_" device="R1206" package3d_urn="urn:adsk.eagle:package:23540/2" value="1M"/>
-<part name="R16" library="rcl" library_urn="urn:adsk.eagle:library:334" deviceset="R-EU_" device="R0402" package3d_urn="urn:adsk.eagle:package:23547/3"/>
+<part name="R16" library="rcl" library_urn="urn:adsk.eagle:library:334" deviceset="R-EU_" device="R0402" package3d_urn="urn:adsk.eagle:package:23547/3" value="15k"/>
 <part name="GND37" library="supply1" library_urn="urn:adsk.eagle:library:371" deviceset="GND" device=""/>
 <part name="IC3" library="MIC5504-3.3YM5-TR" library_urn="urn:adsk.eagle:library:13447306" deviceset="MIC5504-3.3YM5-TR" device="" package3d_urn="urn:adsk.eagle:package:13447309/2"/>

Commit message: HW V1.1 fixed 3.3V supply
Connections:
- removed net N$18: C11.1, C12.1, IC2.VDD/VDDA
- net +3V3: now also C11.1, C12.1, IC2.VDD/VDDA
Changed lines of the file:
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@@
-</segment>
-</net>
-<net name="N$18" class="0">
-<segment>
-<pinref part="IC2" gate="G$1" pin="VDD/VDDA"/>
-<wire x1="101.6" y1="101.6" x2="68.58" y2="101.6" width="0.1524" layer="91"/>
-<pinref part="C11" gate="G$1" pin="1"/>
-<wire x1="68.58" y1="101.6" x2="60.96" y2="101.6" width="0.1524" layer="91"/>
-<wire x1="60.96" y1="101.6" x2="60.96" y2="96.52" width="0.1524" layer="91"/>
-<pinref part="C12" gate="G$1" pin="1"/>
-<wire x1="68.58" y1="96.52" x2="68.58" y2="101.6" width="0.1524" layer="91"/>
-<junction x="68.58" y="101.6"/>
 </segment>
 </net>
@@
 <segment>
 <pinref part="IC2" gate="G$1" pin="VREF+"/>
-<wire x1="101.6" y1="104.14" x2="53.34" y2="104.14" width="0.1524" layer="91"/>
+<wire x1="101.6" y1="104.14" x2="60.96" y2="104.14" width="0.1524" layer="91"/>
 <pinref part="C9" gate="G$1" pin="1"/>
+<wire x1="60.96" y1="104.14" x2="53.34" y2="104.14" width="0.1524" layer="91"/>
 <wire x1="53.34" y1="104.14" x2="45.72" y2="104.14" width="0.1524" layer="91"/>
 <wire x1="45.72" y1="104.14" x2="45.72" y2="96.52" width="0.1524" layer="91"/>
@@
 <wire x1="45.72" y1="114.3" x2="45.72" y2="104.14" width="0.1524" layer="91"/>
 <junction x="45.72" y="104.14"/>
+<pinref part="IC2" gate="G$1" pin="VDD/VDDA"/>
+<wire x1="101.6" y1="101.6" x2="68.58" y2="101.6" width="0.1524" layer="91"/>
+<pinref part="C11" gate="G$1" pin="1"/>
+<wire x1="68.58" y1="101.6" x2="60.96" y2="101.6" width="0.1524" layer="91"/>
+<wire x1="60.96" y1="101.6" x2="60.96" y2="96.52" width="0.1524" layer="91"/>
+<pinref part="C12" gate="G$1" pin="1"/>
+<wire x1="68.58" y1="96.52" x2="68.58" y2="101.6" width="0.1524" layer="91"/>
+<junction x="68.58" y="101.6"/>
+<wire x1="60.96" y1="101.6" x2="60.96" y2="104.14" width="0.1524" layer="91"/>
+<junction x="60.96" y="101.6"/>
+<junction x="60.96" y="104.14"/>
 </segment>
 <segment>

Commit message: V1.1 fixed nixie footprint
Other:
- note added: "TODO: Programmerleiste abändern Montagelöcher Zusätzliche Taster hinzufügen V1.1 change log: 3.3V Versorgung richtig angeschlossen Löcher für Röhren kleiner Bestückungsdruck der Röhren angepasst"
Changed lines of the file:
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@@
 <parts>
 <part name="N4" library="Nixie" library_urn="urn:adsk.eagle:library:1509144" deviceset="IN-12" device="-V3" package3d_urn="urn:adsk.eagle:package:1509184/3"/>
-<part name="N3" library="Nixie" library_urn="urn:adsk.eagle:library:1509144" deviceset="IN-12" device="-V3" package3d_urn="urn:adsk.eagle:package:1509184/3" override_package3d_urn="urn:adsk.eagle:package:1509184/9" override_package_urn="urn:adsk.eagle:footprint:1509183/5"/>
+<part name="N3" library="Nixie" library_urn="urn:adsk.eagle:library:1509144" deviceset="IN-12" device="-V3" package3d_urn="urn:adsk.eagle:package:1509184/3" override_package3d_urn="urn:adsk.eagle:package:1509184/9" override_package_urn="urn:adsk.eagle:footprint:1509183/5" override_locally_modified="yes"/>
 <part name="N2" library="Nixie" library_urn="urn:adsk.eagle:library:1509144" deviceset="IN-12" device="-V3" package3d_urn="urn:adsk.eagle:package:1509184/3"/>
-<part name="N1" library="Nixie" library_urn="urn:adsk.eagle:library:1509144" deviceset="IN-12" device="-V3" package3d_urn="urn:adsk.eagle:package:1509184/3" override_package3d_urn="urn:adsk.eagle:package:1509184/6" override_package_urn="urn:adsk.eagle:footprint:1509183/3"/>
+<part name="N1" library="Nixie" library_urn="urn:adsk.eagle:library:1509144" deviceset="IN-12" device="-V3" package3d_urn="urn:adsk.eagle:package:1509184/3" override_package3d_urn="urn:adsk.eagle:package:1509184/6" override_package_urn="urn:adsk.eagle:footprint:1509183/3" override_locally_modified="yes"/>
 <part name="N6" library="Nixie" library_urn="urn:adsk.eagle:library:1509144" deviceset="INS-1" device="" package3d_urn="urn:adsk.eagle:package:1509158/1"/>
 <part name="N5" library="Nixie" library_urn="urn:adsk.eagle:library:1509144" deviceset="INS-1" device="" package3d_urn="urn:adsk.eagle:package:1509158/1"/>
@@
 </nets>
 </sheet>
+<sheet>
+<plain>
+<text x="0" y="0" size="1.778" layer="91">TODO:
+Programmerleiste abändern
+Montagelöcher
+Zusätzliche Taster hinzufügen
+V1.1 change log:
+3.3V Versorgung richtig angeschlossen
+Löcher für Röhren kleiner
+Bestückungsdruck der Röhren angepasst</text>
+</plain>
+<instances>
+</instances>
+<busses>
+</busses>
+<nets>
+</nets>
+</sheet>
 </sheets>
 </schematic>
 </drawing>
 <compatibility>
+<note version="6.3" minversion="6.2.2" severity="warning">
+Since Version 6.2.2 text objects can contain more than one line,
+which will not be processed correctly with this version.
+</note>
 <note version="8.2" severity="warning">
 Since Version 8.2, EAGLE supports online libraries. The ids

Commit message: Zwischenstand zu V1.1 Revision
Parts:
- added S3: (no value), Wurth_Elektronik_Electromechanic_Switch_rev18c:434121050816
- added SV1: (no value), con-lstb:MA03-1
Connections:
- removed net SWO: J3.4
- new net S3: IC2.PF1-OSC_OUT
- net +3V3: no longer J3.1
- net GND: now also S3.2
- net NRST: no longer J3.5
Changed lines of the file:
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@@
 <part name="GND41" library="supply1" library_urn="urn:adsk.eagle:library:371" deviceset="GND" device=""/>
 <part name="J3" library="EAGLE-BOARD-TO-BOARD_CONNECTORS-rev16c" library_urn="urn:adsk.eagle:library:1555131" deviceset="62100621021" device="" package3d_urn="urn:adsk.eagle:package:1555134/2"/>
-<part name="+3V3" library="supply1" library_urn="urn:adsk.eagle:library:371" deviceset="+3V3" device=""/>
 <part name="GND44" library="supply1" library_urn="urn:adsk.eagle:library:371" deviceset="GND" device=""/>
 <part name="GND43" library="supply1" library_urn="urn:adsk.eagle:library:371" deviceset="GND" device=""/>
+<part name="S3" library="Wurth_Elektronik_Electromechanic_Switch_rev18c" library_urn="urn:adsk.eagle:library:490197" deviceset="434121050816" device="" package3d_urn="urn:adsk.eagle:package:3097884/2" override_package3d_urn="urn:adsk.eagle:package:13439559/2" override_package_urn="urn:adsk.eagle:footprint:3097617/2"/>
+<part name="SV1" library="con-lstb" library_urn="urn:adsk.eagle:library:162" deviceset="MA03-1" device="" package3d_urn="urn:adsk.eagle:package:8339/1"/>
 </parts>
 <sheets>
@@
 <attribute name="VALUE" x="180.34" y="68.58" size="1.27" layer="95"/>
 </instance>
-<instance part="+3V3" gate="G$1" x="172.72" y="83.82" smashed="yes">
-<attribute name="VALUE" x="170.18" y="78.74" size="1.778" layer="96" rot="R90"/>
-</instance>
 <instance part="GND44" gate="1" x="172.72" y="68.58" smashed="yes">
 <attribute name="VALUE" x="170.18" y="66.04" size="1.778" layer="96"/>
+</instance>
+<instance part="S3" gate="G$1" x="38.1" y="25.4" smashed="yes">
+<attribute name="NAME" x="34.29" y="28.956" size="1.778" layer="95"/>
+<attribute name="VALUE" x="33.02" y="22.352" size="1.778" layer="96"/>
+</instance>
+<instance part="SV1" gate="G$1" x="210.82" y="73.66" smashed="yes">
+<attribute name="VALUE" x="209.55" y="66.04" size="1.778" layer="96"/>
+<attribute name="NAME" x="209.55" y="79.502" size="1.778" layer="95"/>
 </instance>
 </instances>
@@
 <wire x1="48.26" y1="40.64" x2="48.26" y2="33.02" width="0.1524" layer="91"/>
 <pinref part="S2" gate="G$1" pin="2"/>
-<wire x1="48.26" y1="33.02" x2="48.26" y2="22.86" width="0.1524" layer="91"/>
+<wire x1="48.26" y1="33.02" x2="48.26" y2="25.4" width="0.1524" layer="91"/>
+<wire x1="48.26" y1="25.4" x2="48.26" y2="22.86" width="0.1524" layer="91"/>
 <wire x1="45.72" y1="33.02" x2="48.26" y2="33.02" width="0.1524" layer="91"/>
 <junction x="48.26" y="33.02"/>
 <pinref part="S1" gate="G$1" pin="1"/>
 <wire x1="45.72" y1="40.64" x2="48.26" y2="40.64" width="0.1524" layer="91"/>
+<pinref part="S3" gate="G$1" pin="2"/>
+<wire x1="45.72" y1="25.4" x2="48.26" y2="25.4" width="0.1524" layer="91"/>
+<junction x="48.26" y="25.4"/>
 </segment>
 <segment>
@@
 <wire x1="83.82" y1="91.44" x2="83.82" y2="88.9" width="0.1524" layer="91"/>
 <label x="83.82" y="91.44" size="1.778" layer="95" rot="MR0"/>
-</segment>
-<segment>
-<pinref part="J3" gate="G$1" pin="5"/>
-<wire x1="190.5" y1="76.2" x2="193.04" y2="76.2" width="0.1524" layer="91" style="longdash"/>
-<label x="193.04" y="76.2" size="1.27" layer="95" xref="yes"/>
 </segment>
 </net>
@@
 <junction x="226.06" y="114.3"/>
 </segment>
-<segment>
-<pinref part="J3" gate="G$1" pin="1"/>
-<wire x1="175.26" y1="78.74" x2="172.72" y2="78.74" width="0.1524" layer="91" style="longdash"/>
-<wire x1="172.72" y1="78.74" x2="172.72" y2="81.28" width="0.1524" layer="91" style="longdash"/>
-<pinref part="+3V3" gate="G$1" pin="+3V3"/>
-</segment>
 </net>
 <net name="+5V" class="0">
@@
 </segment>
 </net>
-<net name="SWO" class="0">
-<segment>
-<pinref part="J3" gate="G$1" pin="4"/>
-<wire x1="190.5" y1="73.66" x2="193.04" y2="73.66" width="0.1524" layer="91" style="longdash"/>
-<label x="193.04" y="73.66" size="1.27" layer="95" xref="yes"/>
-</segment>
-</net>
 <net name="FB_170V" class="0">
 <segment>
@@
 </segment>
 </net>
+<net name="S3" class="0">
+<segment>
+<label x="99.06" y="93.98" size="1.778" layer="95" rot="MR0"/>
+<pinref part="IC2" gate="G$1" pin="PF1-OSC_OUT"/>
+<wire x1="101.6" y1="93.98" x2="91.44" y2="93.98" width="0.1524" layer="91"/>
+</segment>
+</net>
